File: mcu.kicad_sch (KiCad schematic)
At the start: 54 parts, among them J1 Conn_01x05, J10 Conn_01x02_Pin, J11 Ext_Tamper, J4 USB_B_Micro, J5 Conn_01x01_Pin, J6 Conn_01x01_Pin, J7 Conn_01x01_Pin, J8 Conn_01x01_Pin, J9 Conn_Coaxial, Q2 DMP3056, Q3 2N7002, SW1 SW_Push, U1 STM32G473CCUx, U10 NEO-6M, U12 AT24CS32-XHM, Y1 8 MHz, Y2 ECS-.327-12.5-34QCS-TR

Commit message: end of day commit
Parts:
- added C52: 100n, Capacitor_SMD:C_0603_1608Metric_Pad1.08x0.95mm_HandSolder, symbol Device:C_Small
- added D6: Blue, LED_SMD:LED_0805_2012Metric, symbol Device:LED_Small
- added R52: 3k3, Resistor_SMD:R_0603_1608Metric_Pad0.98x0.95mm_HandSolder, symbol Device:R_Small
- C47: footprint Capacitor_SMD:C_0603_1608Metric_Pad1.08x0.95mm_HandSolder -> Capacitor_SMD:C_0805_2012Metric_Pad1.18x1.45mm_HandSolder
Connections:
- net GP4_IN_OUT_ACC8 is gone; now on net EXP_BD_REQ: U1.30 (PA8)
- net GND: now also C52.1, D6.1 (K)
- net TIMEPULSE: now reaches U10.3 (TIMEPULSE)
- net TIMEPULSE: now also U1.25 (PB12), R52.1
- net at U1.20 (VREF+): now also C52.2
- net RDY: now reaches U1.43 (PB5)
- new net: D6.2 (A), R52.2
- no-connect marks 9 -> 8
Other:
- note added: "3v3 pins"
