File: micro17.kicad_pcb (KiCad board)
At the start: 4 copper layers, 60 x 71 mm, 144 parts, among them J1 Conn_01x05, J10 Conn_01x02_Pin, J11 Ext_Tamper, J2 Conn_01x40_Pin, J5 Conn_01x01_Pin, J6 Conn_01x01_Pin, J7 Conn_01x01_Pin, J8 Conn_01x01_Pin, J9 Conn_Coaxial, Q2 DMP3056, Q3 2N7002, SW1 SW_Push, U1 STM32G473CCUx, U10 NEO-6M, U11 TXS0108EPW, U12 AT24CS32-XHM, U13 XC6220B331MR, U2 XC6220B331MR, U4 MCP6002, U5 MCP4451-503-ST, U6 MCP6002, U7 MCP6002, U9 LMR14206, Y1 8 MHz, Y2 ECS-.327-12.5-34QCS-TR

Commit message: end of day commit
Parts:
- added C52: 100n, Capacitor_SMD:C_0603_1608Metric_Pad1.08x0.95mm_HandSolder, F.Cu at (203.3, 98.2)
- added D6: Blue, LED_SMD:LED_0805_2012Metric, F.Cu at (146.5, 121.2)
- added Q4: BC817, Package_TO_SOT_SMD:SOT-23, F.Cu at (204.2, 103.1)
- added Q5: BC817, Package_TO_SOT_SMD:SOT-23, F.Cu at (204.2, 107.7)
- added R25: 3k3, Resistor_SMD:R_0603_1608Metric_Pad0.98x0.95mm_HandSolder, F.Cu at (168.6, 104.6)
- added R45: 3k3, Resistor_SMD:R_0603_1608Metric_Pad0.98x0.95mm_HandSolder, F.Cu at (153.7, 95.6)
- added R46: 3k3, Resistor_SMD:R_0603_1608Metric_Pad0.98x0.95mm_HandSolder, F.Cu at (167.9, 94.1)
- added R47: 3k3, Resistor_SMD:R_0603_1608Metric_Pad0.98x0.95mm_HandSolder, F.Cu at (200.4, 102.1)
- added R48: 3k3, Resistor_SMD:R_0603_1608Metric_Pad0.98x0.95mm_HandSolder, F.Cu at (152.9, 92.8)
- added R49: 3k3, Resistor_SMD:R_0603_1608Metric_Pad0.98x0.95mm_HandSolder, F.Cu at (200.3, 106.7)
- added R50: 3k3, Resistor_SMD:R_0603_1608Metric_Pad0.98x0.95mm_HandSolder, F.Cu at (160.1, 87.2)
- added R51: 3k3, Resistor_SMD:R_0603_1608Metric_Pad0.98x0.95mm_HandSolder, F.Cu at (160.1, 89.6)
- added R52: 3k3, Resistor_SMD:R_0603_1608Metric_Pad0.98x0.95mm_HandSolder, F.Cu at (151.6, 117.9)
- added R53: 3k3, Resistor_SMD:R_0603_1608Metric_Pad0.98x0.95mm_HandSolder, F.Cu at (164.8, 87.2)
- added TP3: GP, TestPoint:TestPoint_Pad_D1.0mm, F.Cu at (173.7, 113.2)
- added TP4: GP, TestPoint:TestPoint_Pad_D1.0mm, F.Cu at (173.7, 111.1)
- added U3: CPC1117N, Package_SO:SOP-4_3.8x4.1mm_P2.54mm, F.Cu at (170.0, 110.4)
- C47: footprint Capacitor_SMD:C_0603_1608Metric_Pad1.08x0.95mm_HandSolder -> Capacitor_SMD:C_0805_2012Metric_Pad1.18x1.45mm_HandSolder
- TP6: moved to B.Cu
- moved TP6 54.8 mm to (135.2, 83.2), turned to 180 degrees
- moved SYM1 14.5 mm to (138.3, 55.9), turned to 0 degrees
- moved TP10 1.79 mm to (166.1, 91.0)
- moved TP7 1.70 mm to (168.2, 91.0)
- moved TP2 1.38 mm to (151.4, 82.8)
- moved C34 1.32 mm to (152.0, 80.5)
- moved C15 1.22 mm to (154.6, 79.5)
- moved C47 1.19 mm to (171.5, 91.5)
- moved C18 1.15 mm to (156.2, 79.5)
- moved BT1 1.14 mm to (177.4, 100.6)
- moved R42 1.00 mm to (172.9, 88.6)
- moved R7 1.00 mm to (154.6, 83.4)
- moved R9 1.00 mm to (156.1, 83.4)
- moved C51 0.97 mm to (150.0, 117.9)
- moved C20 0.96 mm to (159.1, 83.5)
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Connections:
- R31 pad 1: EXP1_CS -> EXP1_CS_5V
- R31 pad 2: EXP1_CS_5V -> EXP1_CS
- U1 pad 20: unconnected-(U1-VREF+-Pad20) -> Net-(U1-VREF+)
- U1 pad 25: unconnected-(U1-PB12-Pad25) -> TIMEPULSE
- U1 pad 30: unconnected-(U1-PA8-Pad30) -> EXP_BD_REQ
- U1 pad 43: unconnected-(U1-PB5-Pad43) -> RDY
- U10 pad 3: unconnected-(U10-TIMEPULSE-Pad3) -> TIMEPULSE
- U11 pad 6: GP4_IN_OUT_ACC8 -> AUDIO_OUT_MUTE
- U11 pad 8: AUDIO_OUT_MUTE -> RDY
Routing:
- net EXP_BD_REQ: track 1.29 -> 27.4 mm, vias 1 -> 3
- net RDY: track 0.00 -> 23.0 mm, vias 0 -> 2
- net BASEBAND_BYPASS: track 2.64 -> 22.2 mm, vias 1 -> 3
- net CH_Activity_5V: track 19.6 -> 36.1 mm, vias 1 -> 2
- net MCU_RX: track 20.0 -> 33.7 mm, vias 2 -> 4
- net +BATT: track 82.3 -> 91.8 mm
- net +3V3: track 46.8 -> 38.2 mm, vias 10 -> 11
- net GND: track 6.57 -> 14.6 mm, vias 26 -> 38
- net +5V: track 148.5 -> 140.8 mm, vias 11 -> 12
- net TIMEPULSE: track 0.00 -> 7.15 mm, vias 0 -> 1
- net Net-(TP4-Pad1): track 0.00 -> 5.82 mm
- net Net-(D6-A): track 0.00 -> 5.73 mm
- net Net-(R25-Pad2): track 0.00 -> 3.72 mm
- net OPT_CS: track 12.1 -> 15.6 mm
- net OPT_CS_5V: track 7.33 -> 10.6 mm
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Other:
- board text added: "+-"
- board text added: "3v3 Rst SWC SWD Gnd"
- board text added: "5V Gnd"
- board text added: "Txo Rxi"
