File: fltrs.kicad_sch (KiCad schematic)
At the start: 55 parts, among them U3 CPC1117N, U4 MCP6002, U5 MCP4451-503-ST, U6 MCP6002, U7 MCP6002

Commit message: V1.0 Final touch
Other:
- moved on the sheet: R17, R20
Changed lines of the file:
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@@
 	(wire
 		(pts
-			(xy 158.75 160.02) (xy 158.75 163.195)
+			(xy 158.75 161.29) (xy 158.75 163.195)
 		)
 		(stroke
@@
 	(wire
 		(pts
-			(xy 148.59 149.225) (xy 148.59 155.575)
+			(xy 148.59 149.225) (xy 148.59 156.21)
 		)
 		(stroke
@@
 	(wire
 		(pts
-			(xy 148.59 160.655) (xy 148.59 163.195)
+			(xy 148.59 161.29) (xy 148.59 163.195)
 		)
 		(stroke
@@
 		(on_board yes)
 		(dnp no)
-		(fields_autoplaced yes)
 		(property "Reference" "C26"
-			(at 121.92 172.8089 0)
+			(at 122.174 173.99 0)
 			(effects
 				(font
@@
 		)
 		(property "Value" "22u"
-			(at 121.92 175.3489 0)
+			(at 122.174 176.276 0)
 			(effects
 				(font
@@
 	(symbol
 		(lib_id "power:VDDA")
-		(at 158.75 154.94 0)
+		(at 158.75 156.21 0)
 		(unit 1)
 		(exclude_from_sim no)
@@
 		(fields_autoplaced yes)
 		(property "Reference" "#PWR082"
-			(at 158.75 158.75 0)
+			(at 158.75 160.02 0)
 			(effects
 				(font
@@
 		)
 		(property "Value" "VDDA"
-			(at 158.75 149.86 0)
+			(at 158.75 151.13 0)
 			(effects
 				(font
@@
 		)
 		(property "Footprint" ""
-			(at 158.75 154.94 0)
+			(at 158.75 156.21 0)
 			(effects
 				(font
@@
 		)
 		(property "Datasheet" ""
-			(at 158.75 154.94 0)
+			(at 158.75 156.21 0)
 			(effects
 				(font
@@
 		)
 		(property "Description" "Power symbol creates a global label with name \"VDDA\""
-			(at 158.75 154.94 0)
+			(at 158.75 156.21 0)
 			(effects
 				(font
@@
 	(symbol
 		(lib_id "Device:R_Small")
-		(at 158.75 157.48 0)
+		(at 158.75 158.75 0)
 		(unit 1)
 		(exclude_from_sim no)
@@
 		(fields_autoplaced yes)
 		(property "Reference" "R20"
-			(at 161.29 156.21 0)
+			(at 161.29 157.48 0)
 			(effects
 				(font
@@
 		)
 		(property "Value" "22k"
-			(at 161.29 158.75 0)
+			(at 161.29 160.02 0)
 			(effects
 				(font
@@
 		)
 		(property "Footprint" "Resistor_SMD:R_0402_1005Metric"
-			(at 158.75 157.48 0)
+			(at 158.75 158.75 0)
 			(effects
 				(font
@@
 		)
 		(property "Datasheet" ""
-			(at 158.75 157.48 0)
+			(at 158.75 158.75 0)
 			(effects
 				(font
@@
 		)
 		(property "Description" ""
-			(at 158.75 157.48 0)
+			(at 158.75 158.75 0)
 			(effects
 				(font
@@
 		)
 		(property "MPN" "C2909337"
-			(at 158.75 157.48 0)
+			(at 158.75 158.75 0)
 			(effects
 				(font
@@
 		)
 		(property "Height" ""
-			(at 158.75 157.48 0)
+			(at 158.75 158.75 0)
 			(effects
 				(font
@@
 		)
 		(property "Manufacturer_Name" ""
-			(at 158.75 157.48 0)
+			(at 158.75 158.75 0)
 			(effects
 				(font
@@
 		)
 		(property "Manufacturer_Part_Number" ""
-			(at 158.75 157.48 0)
+			(at 158.75 158.75 0)
 			(effects
 				(font
@@
 		)
 		(property "Mouser Part Number" ""
-			(at 158.75 157.48 0)
+			(at 158.75 158.75 0)
 			(effects
 				(font
@@
 		)
 		(property "Mouser Price/Stock" ""
-			(at 158.75 157.48 0)
+			(at 158.75 158.75 0)
 			(effects
 				(font
@@
 		)
 		(property "LCSC" "C2909337"
-			(at 158.75 157.48 0)
+			(at 158.75 158.75 0)
 			(effects
 				(font
@@
 		)
 		(property "JLC" ""
-			(at 158.75 157.48 0)
+			(at 158.75 158.75 0)
 			(effects
 				(font
@@
 		)
 		(property "PN" ""
-			(at 158.75 157.48 0)
+			(at 158.75 158.75 0)
 			(effects
 				(font
@@
 	(symbol
 		(lib_id "Device:R_Small")
-		(at 148.59 158.115 0)
+		(at 148.59 158.75 0)
 		(unit 1)
 		(exclude_from_sim no)
@@
 		(fields_autoplaced yes)
 		(property "Reference" "R17"
-			(at 151.13 156.845 0)
+			(at 151.13 157.48 0)
 			(effects
 				(font
@@
 		)
 		(property "Value" "22k"
-			(at 151.13 159.385 0)
+			(at 151.13 160.02 0)
 			(effects
 				(font
@@
 		)
 		(property "Footprint" "Resistor_SMD:R_0402_1005Metric"
-			(at 148.59 158.115 0)
+			(at 148.59 158.75 0)
 			(effects
 				(font
@@
 		)
 		(property "Datasheet" ""
-			(at 148.59 158.115 0)
+			(at 148.59 158.75 0)
 			(effects
 				(font
@@
 		)
 		(property "Description" ""
-			(at 148.59 158.115 0)
+			(at 148.59 158.75 0)
 			(effects
 				(font
@@
 		)
 		(property "MPN" "C2909337"
-			(at 148.59 158.115 0)
+			(at 148.59 158.75 0)
 			(effects
 				(font
@@
 		)
 		(property "Height" ""
-			(at 148.59 158.115 0)
+			(at 148.59 158.75 0)
 			(effects
 				(font
@@
 		)
 		(property "Manufacturer_Name" ""
-			(at 148.59 158.115 0)
+			(at 148.59 158.75 0)
 			(effects
 				(font
@@
 		)
 		(property "Manufacturer_Part_Number" ""
-			(at 148.59 158.115 0)
+			(at 148.59 158.75 0)
 			(effects
 				(font
@@
 		)
 		(property "Mouser Part Number" ""
-			(at 148.59 158.115 0)
+			(at 148.59 158.75 0)
 			(effects
 				(font
@@
 		)
 		(property "Mouser Price/Stock" ""
-			(at 148.59 158.115 0)
+			(at 148.59 158.75 0)
 			(effects
 				(font
@@
 		)
 		(property "LCSC" "C2909337"
-			(at 148.59 158.115 0)
+			(at 148.59 158.75 0)
 			(effects
 				(font
@@
 		)
 		(property "JLC" ""
-			(at 148.59 158.115 0)
+			(at 148.59 158.75 0)
 			(effects
 				(font
@@
 		)
 		(property "PN" ""
-			(at 148.59 158.115 0)
+			(at 148.59 158.75 0)
 			(effects
 				(font
@@
 		(on_board yes)
 		(dnp no)
-		(fields_autoplaced yes)
 		(property "Reference" "C28"
-			(at 151.13 166.4589 0)
+			(at 150.876 166.878 0)
 			(effects
 				(font
@@
 		)
 		(property "Value" "22u"
-			(at 151.13 168.9989 0)
+			(at 151.13 169.418 0)
 			(effects
 				(font
@@
 		(on_board yes)
 		(dnp no)
-		(fields_autoplaced yes)
 		(property "Reference" "R21"
-			(at 161.29 167.005 0)
+			(at 161.29 166.878 0)
 			(effects
 				(font
